File: NearFi.kicad_pcb (KiCad board)
At the start: 2 copper layers, 45.6 x 45.6 mm, 21 parts, among them J1 PWR_CONN, J2 CONN_PROG, SW1 RESET, SW2 BOOT, U1 ESP32-S2-WROVER, U2 TLV1117-33

Commit message: Modified PCB
Parts:
- turned C1 to 90 degrees
Routing:
- net +3V3: track 96.8 -> 95.7 mm, vias 15 -> 14
- net GND: track 3.36 -> 4.49 mm, vias 67 -> 68
- net /RGB: track 16.2 -> 15.2 mm
