File: bitec_nearfi_pcb.kicad_pcb (KiCad board)
At the start: 2 copper layers, 45.6 x 45.6 mm, 21 parts, among them J1 PWR_CONN, J2 CONN_PROG, SW1 RESET, SW2 BOOT, U1 ESP32-S2-WROVER, U2 TLV1117-33

Commit message: Finished version 1
Parts:
- added BZ1: Buzzer, Buzzer_Beeper:Buzzer_Murata_PKMCS0909E4000-R1, F.Cu at (133.3, 67.6)
- added Q1: MMBT3904, Package_TO_SOT_SMD:SOT-23, F.Cu at (130.8, 61.0)
- added R2: 10K, Resistor_SMD:R_0805_2012Metric_Pad1.20x1.40mm_HandSolder, F.Cu at (136.1, 61.0)
- moved D2 4.50 mm to (133.3, 74.4), turned to 0 degrees
- moved R3 0.51 mm to (142.5, 74.4)
Connections:
- U1 pad 11: (no net) -> /BUZZER
Routing:
- net Net-(BZ1-Pad2): track 0.00 -> 10.8 mm
- net +3V3: track 95.7 -> 102.4 mm, vias 14 -> 15
- net /BUZZER: track 0.00 -> 5.14 mm
- net Net-(Q1-Pad1): track 0.00 -> 3.80 mm
- net GND: vias 68 -> 66
Other:
- board text added: "Name: NearFi Author: Mauricio Barroso Date: 17/05/21 Version: 1.0 Rev: 2"
- board text removed: "Name: natFi Author: Mauricio Barroso Date: 14/05/21 Version: 1.0 Rev: 2"
