File: bitec_nearfi_pcb.sch (KiCad schematic (older format))
At the start: 21 parts, among them J1 PWR_CONN, J2 CONN_PROG, SW1 RESET, SW2 BOOT, U1 ESP32-S2-WROVER, U2 TLV1117-33

Commit message: Finished version 1
Parts:
- added BZ1: Buzzer, Buzzer_Beeper:Buzzer_Murata_PKMCS0909E4000-R1, symbol Device:Buzzer
- added Q1: MMBT3904, Package_TO_SOT_SMD:SOT-23, symbol Transistor_BJT:MMBT3904
- added R2: 10K, Resistor_SMD:R_0805_2012Metric_Pad1.20x1.40mm_HandSolder, symbol Device:R_Small
Connections:
- net +3V3: now also BZ1.1 (-)
- net GND: now also Q1.2 (E)
- net BUZZER: now reaches U1.11 (IO08)
- net BUZZER: now also R2.1
- new net: BZ1.2 (+), Q1.3 (C)
- new net: Q1.1 (B), R2.2
- no-connect marks 37 -> 36
Other:
- note added: "BUZZER"
- note added: "Connectors"
- moved on the sheet: C1, C10, C5, C6, C7, D1, D2, H1, H2, H3, H4, J1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
